File: Feather M0 Temp Sensor/Feather M0 Temp Sensor.kicad_sch (KiCad schematic)
At the start: 3 parts, among them J1 Feather_Long_Side, J2 Feather_Short_Side, U1 Adafruit_SHT4x

Commit message: Saved files
Parts:
- J1: footprint Connector_PinSocket_2.54mm:PinSocket_1x15_P2.54mm_Vertical -> Connector_PinSocket_2.54mm:PinSocket_1x13_P2.54mm_Vertical
Changed lines of the file:
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@@
     (property "Reference" "J1" (id 0) (at 76.2 100.33 90))
     (property "Value" "Feather_Long_Side" (id 1) (at 78.74 100.33 90))
-    (property "Footprint" "Connector_PinSocket_2.54mm:PinSocket_1x15_P2.54mm_Vertical" (id 2) (at 82.55 100.33 0)
+    (property "Footprint" "Connector_PinSocket_2.54mm:PinSocket_1x13_P2.54mm_Vertical" (id 2) (at 82.55 100.33 0)
       (effects (font (size 1.27 1.27)) hide)
     )
@@
   (symbol_instances
     (path "/a13aaac4-75bf-45e4-a42f-e0c4642f65e3"
-      (reference "J1") (unit 1) (value "Feather_Long_Side") (footprint "Connector_PinSocket_2.54mm:PinSocket_1x15_P2.54mm_Vertical")
+      (reference "J1") (unit 1) (value "Feather_Long_Side") (footprint "Connector_PinSocket_2.54mm:PinSocket_1x13_P2.54mm_Vertical")
     )
     (path "/fabdb2e1-04b0-4ef0-a2ca-215d68d896f1"
